Commit message: planning OMPL modificado en ur5_moveit_config

File: ur_ws/src/ur5_moveit_config/config/ur5_full.ros2_control.xacro (robot description, xacro)
@@ -8,18 +8,4 @@
                 <plugin>mock_components/GenericSystem</plugin>
             </hardware>
-            <joint name="robotiq_hande_left_finger_joint">
-                <command_interface name="position"/>
-                <state_interface name="position">
-                  <param name="initial_value">${initial_positions['robotiq_hande_left_finger_joint']}</param>
-                </state_interface>
-                <state_interface name="velocity"/>
-            </joint>
-            <joint name="robotiq_hande_right_finger_joint">
-                <command_interface name="position"/>
-                <state_interface name="position">
-                  <param name="initial_value">${initial_positions['robotiq_hande_right_finger_joint']}</param>
-                </state_interface>
-                <state_interface name="velocity"/>
-            </joint>
             <joint name="shoulder_pan_joint">
                 <command_interface name="position"/>
